Commit message: Updated URDF and launch files

File: description/robot.urdf (robot description, URDF)
Before this commit: robot fire_robot, 4 links, 3 joints
Links:
- link base_link: mass None -> 0.5; geometry collision box size=0.14 0.14 0.009; visual box size=0.14 0.14 0.009
- link laser_frame: mass None -> 0.05; geometry collision cylinder length=0.04 radius=0.03; visual cylinder length=0.04 radius=0.03
- link left_wheel: mass None -> 0.05; geometry collision cylinder length=0.015 radius=0.0215; visual cylinder length=0.015 radius=0.0215
- link right_wheel: mass None -> 0.05; geometry collision cylinder length=0.015 radius=0.0215; visual cylinder length=0.015 radius=0.0215

Commit message: Fix duplicate package, add hardware-free sim test rig, fix TF tree and URDF bugs
- Remove committed build/install/log artifacts, restore proper .gitignore
- Fix fire_bridge.py silent failure when serial connection unavailable
- Add collision/inertial tags to URDF links
- Add base_footprint root link, fix odom TF parent conflict
- Add joint_state_publisher to launch file
- Add sim_bridge.py for hardware-free odometry testing
- Add drive_test_monitor.py and rotation_test_monitor.py for automated
  odometry validation (straight-line: -0.5% error, rotation: 0.1% error)
- Add fake_scan.py for testing LaserScan/SLAM wiring without LIDAR hardware

File: description/robot.urdf (robot description, URDF)
Before this commit: robot fire_robot, 4 links, 3 joints
Links:
- added link base_footprint
Joints:
- added joint base_footprint_to_base_link: type fixed, parent base_footprint, child base_link, origin xyz=0 0 0 rpy=0 0 0
